File: StrainGageAmpSMD.sch (EAGLE design)
At the start: 55 parts

Commit message: Reduced from 6 channels to 3
-Reduced 6 channels to 3
-Changed all resistors to 0603 format
Parts:
- removed LM1, LM2, LM324: QUAD_OPAMPD, adafruit:QUAD_OPAMPD
- removed O0, O1, O2: 22-23-2021, con-molex:22-23-2021
- removed R10, R11, R17, R18, R4, R5: 2.2k, adafruit:R-US_R1206
- removed R12, R13, R14, R19, R20, R21, R6, R7, R8: 352, adafruit:R-US_R0603
- removed R15, R16, R2, R22, R3, R9: 560k, adafruit:R-US_R1206
- removed RTANGLE: 22-23-2081, con-molex:22-23-2081
- added GND_VCC_0_1_2: 22-23-2051, con-molex:22-23-2051
- R1: device adafruit:R-US_R1206 -> rcl:R-US_R0603
- R23, R24, R25, R29, R30, R31, R32, R36, R37, R38, R39: device adafruit:R-US_R1206 -> adafruit:R-US_R0603
Connections:
- removed net N$1: LM1A.+IN, R12.2, R13.1
- removed net N$10: LM1B.+IN, O1-1.S, R14.1
- removed net N$11: LM1A.-IN, LM1A.OUT, R10.1
- removed net N$12: LM1B.-IN, LM1B.OUT, R11.1
- removed net N$13: LM1C.-IN, R11.2, R9.1
- removed net N$14: LM1C.+IN, R1.1, R10.2
- removed net N$15: LM2A.+IN, R19.2, R20.1
- removed net N$16: LM2B.+IN, O2-1.S, R21.1
- removed net N$17: LM2A.-IN, LM2A.OUT, R17.1
- removed net N$18: LM2B.-IN, LM2B.OUT, R18.1
- removed net N$19: LM2C.-IN, R16.1, R18.2
- removed net N$2: LM324A.+IN, R6.2, R7.1
- removed net N$20: LM2C.+IN, R15.1, R17.2
- removed net N$3: LM324B.+IN, O0-1.S, R8.1
- removed net N$4: LM324A.-IN, LM324A.OUT, R4.1
- removed net N$5: LM324B.-IN, LM324B.OUT, R5.1
- removed net N$6: LM324C.-IN, R3.1, R5.2
- removed net N$7: LM324C.+IN, R2.1, R4.2
- removed net N$8: LM324C.OUT, R3.2, RTANGLE-6.S
- removed net N$81: LM1C.OUT, R9.2, RTANGLE-5.S
- removed net N$82: LM2C.OUT, R16.2, RTANGLE-4.S
- net GND: now also GND_VCC_0_1_2-5.S; no longer LM1P.V-, LM2P.V-, LM324P.V-, O0-2.S, O1-2.S, O2-2.S, R12.1, R15.2, R19.1, R2.2, R22.2, R6.1, RTANGLE-8.S
- net N$26: now also R1.1; no longer R22.1
- net N$83: now also GND_VCC_0_1_2-1.S; no longer RTANGLE-3.S
- net N$84: now also GND_VCC_0_1_2-2.S; no longer RTANGLE-2.S
- net N$85: now also GND_VCC_0_1_2-3.S; no longer RTANGLE-1.S
- net VCC: now also GND_VCC_0_1_2-4.S; no longer LM1P.V+, LM2P.V+, LM324P.V+, R13.2, R14.2, R20.2, R21.2, R7.2, R8.2, RTANGLE-7.S
Other:
- moved on the sheet: R1
